File: button-matrix.sch (KiCad schematic (older format))
At the start: 74 parts, among them SW1 TL1105, SW10 TL1105, SW11 TL1105, SW12 TL1105, SW13 TL1105, SW14 TL1105, SW15 TL1105, SW16 TL1105, SW17 TL1105, SW18 TL1105, SW2 TL1105, SW20 TL1105, SW21 TL1105, SW22 TL1105, SW23 TL1105, SW24 TL1105, SW25 TL1105, SW26 TL1105, SW27 TL1105, SW28 TL1105, SW29 TL1105, SW3 TL1105, SW30 TL1105, SW31 TL1105, SW32 TL1105, SW33 TL1105, SW34 TL1105, SW35 TL1105, SW36 TL1105, SW37 TL1105, SW38 TL1105, SW39 TL1105, SW4 TL1105, SW5 TL1105, SW6 TL1105, SW7 TL1105, SW9 TL1105

Commit message: Added JCLC part numbers.
Parts:
- D10, D11, D12, D13, D14, D15, D16, D17, D18, D19, D20, D21, D22, D23, D24, D25, D26, D27, D28, D29, D30, D31, D32, D33, D34, D35, D36, D37, D38, D39, D40, D41, D5, D6, D8, D9: symbol Device:D -> sequencer-rescue:D-Device
- D7: symbol Device:D -> sequencer-rescue:D-Device; LCSC (none) -> C81598
Changed lines of the file:
@@
 EESchema Schematic File Version 4
 LIBS:sequencer-cache
-EELAYER 26 0
+EELAYER 30 0
 EELAYER END
 $Descr A4 11693 8268
@@
 $EndComp
 $Comp
-L Device:D D7
+L sequencer-rescue:D-Device D7
 U 1 1 59D9507A
 P 2400 1650
@@
 F 5 "1N4148W-7-F" H 2400 1850 50  0001 C CNN "MFP"
 F 6 "SOD-123" H 2400 1850 50  0001 C CNN "Package"
+F 7 "C81598" H 2400 1650 50  0001 C CNN "LCSC"
 	1    2400 1650
 	0    -1   -1   0
 $EndComp
 $Comp
-L Device:D D5
+L sequencer-rescue:D-Device D5
 U 1 1 59D950D5
 P 2400 2350
@@
 $EndComp
 $Comp
-L Device:D D14
+L sequencer-rescue:D-Device D14
 U 1 1 59D9524B
 P 2400 3050
@@
 $EndComp
 $Comp
-L Device:D D24
+L sequencer-rescue:D-Device D24
 U 1 1 59D952C4
 P 2400 3750
@@
 $EndComp
 $Comp
-L Device:D D33
+L sequencer-rescue:D-Device D33
 U 1 1 59D952CD
 P 2400 4450
@@
 $EndComp
 $Comp
-L Device:D D8
+L sequencer-rescue:D-Device D8
 U 1 1 59D955C1
 P 3300 1650
@@
 $EndComp
 $Comp
-L Device:D D6
+L sequencer-rescue:D-Device D6
 U 1 1 59D955C7
 P 3300 2350
@@
 $EndComp
 $Comp
-L Device:D D15
+L sequencer-rescue:D-Device D15
 U 1 1 59D955D0
 P 3300 3050
@@
 $EndComp
 $Comp
-L Device:D D25
+L sequencer-rescue:D-Device D25
 U 1 1 59D955D9
 P 3300 3750
@@
 $EndComp
 $Comp
-L Device:D D35
+L sequencer-rescue:D-Device D35
 U 1 1 59D955E2
 P 3300 4450
@@
 $EndComp
 $Comp
-L Device:D D9
+L sequencer-rescue:D-Device D9
 U 1 1 59D95864
 P 4200 1650
@@
 $EndComp
 $Comp
-L Device:D D12
+L sequencer-rescue:D-Device D12
 U 1 1 59D9586A
 P 4200 2350
@@
 $EndComp
 $Comp
-L Device:D D16
+L sequencer-rescue:D-Device D16
 U 1 1 59D95873
 P 4200 3050
@@
 $EndComp
 $Comp
-L Device:D D26
+L sequencer-rescue:D-Device D26
 U 1 1 59D9587C
 P 4200 3750
@@
 $EndComp
 $Comp
-L Device:D D36
+L sequencer-rescue:D-Device D36
 U 1 1 59D95885
 P 4200 4450
@@
 $EndComp
 $Comp
-L Device:D D10
+L sequencer-rescue:D-Device D10
 U 1 1 59D958C3
 P 5100 1650
@@
 $EndComp
 $Comp
-L Device:D D13
+L sequencer-rescue:D-Device D13
 U 1 1 59D958C9
 P 5100 2350
@@
 $EndComp
 $Comp
-L Device:D D17
+L sequencer-rescue:D-Device D17
 U 1 1 59D958D2
 P 5100 3050
@@
 $EndComp
 $Comp
-L Device:D D27
+L sequencer-rescue:D-Device D27
 U 1 1 59D958DB
 P 5100 3750
@@
 $EndComp
 $Comp
-L Device:D D37
+L sequencer-rescue:D-Device D37
 U 1 1 59D958E4
 P 5100 4450
@@
 $EndComp
 $Comp
-L Device:D D11
+L sequencer-rescue:D-Device D11
 U 1 1 59D960A7
 P 6000 1650
@@
 $EndComp
 $Comp
-L Device:D D22
+L sequencer-rescue:D-Device D22
 U 1 1 59D960AD
 P 6000 2350
@@
 $EndComp
 $Comp
-L Device:D D18
+L sequencer-rescue:D-Device D18
 U 1 1 59D960B6
 P 6000 3050
@@
 $EndComp
 $Comp
-L Device:D D28
+L sequencer-rescue:D-Device D28
 U 1 1 59D960BF
 P 6000 3750
@@
 $EndComp
 $Comp
-L Device:D D38
+L sequencer-rescue:D-Device D38
 U 1 1 59D960C8
 P 6000 4450
@@
 $EndComp
 $Comp
-L Device:D D23
+L sequencer-rescue:D-Device D23
 U 1 1 59D96115
 P 6900 2350
@@
 $EndComp
 $Comp
-L Device:D D19
+L sequencer-rescue:D-Device D19
 U 1 1 59D9611E
 P 6900 3050
@@
 $EndComp
 $Comp
-L Device:D D29
+L sequencer-rescue:D-Device D29
 U 1 1 59D96127
 P 6900 3750
@@
 $EndComp
 $Comp
-L Device:D D39
+L sequencer-rescue:D-Device D39
 U 1 1 59D96130
 P 6900 4450
@@
 $EndComp
 $Comp
-L Device:D D34
+L sequencer-rescue:D-Device D34
 U 1 1 59D9617D
 P 7800 2350
@@
 $EndComp
 $Comp
-L Device:D D20
+L sequencer-rescue:D-Device D20
 U 1 1 59D96186
 P 7800 3050
@@
 $EndComp
 $Comp
-L Device:D D30
+L sequencer-rescue:D-Device D30
 U 1 1 59D9618F
 P 7800 3750
@@
 $EndComp
 $Comp
-L Device:D D40
+L sequencer-rescue:D-Device D40
 U 1 1 59D96198
 P 7800 4450
@@
 $EndComp
 $Comp
-L Device:D D32
+L sequencer-rescue:D-Device D32
 U 1 1 59D961E5
 P 8700 2350
@@
 $EndComp
 $Comp
-L Device:D D21
+L sequencer-rescue:D-Device D21
 U 1 1 59D961EE
 P 8700 3050
@@
 $EndComp
 $Comp
-L Device:D D31
+L sequencer-rescue:D-Device D31
 U 1 1 59D961F7
 P 8700 3750
@@
 $EndComp
 $Comp
-L Device:D D41
+L sequencer-rescue:D-Device D41
 U 1 1 59D96200
 P 8700 4450
