File: dac.sch (KiCad schematic (older format))
At the start: 46 parts, among them U15 OPA4172, U4 OPA4172, U8 DAC8568C

Commit message: Added JCLC part numbers.
Parts:
- C11, C12, C15, C16, C25, C26, C27, C28, C29, C3, C33, C34, C37, C38, C4, C47, C48: symbol Device:C -> sequencer-rescue:C-Device
- R22, R23, R24, R25, R28, R29, R34, R35, R41, R42, R43, R48, R51, R52, R53, R54, R56, R57, R59, R60, R62, R63, R64, R65: symbol Device:R -> sequencer-rescue:R-Device
- R44: symbol Device:R -> sequencer-rescue:R-Device; LCSC (none) -> C23352
- R47: symbol Device:R -> sequencer-rescue:R-Device; LCSC (none) -> C31850
- U15, U4: symbol Amplifier_Operational:OPA4134 -> sequencer-rescue:OPA4134-Amplifier_Operational
