File: global.sch (KiCad schematic (older format))
At the start: 37 parts, among them Q5 MMBT3904, U11 74HC165, U12 74HC595, U13 74HC595, U14 74HC595, U5 74HCT125

Commit message: Added JCLC part numbers.
Parts:
- C43, C44, C45, C49: symbol Device:C -> sequencer-rescue:C-Device
- C6: symbol Device:C -> sequencer-rescue:C-Device; LCSC (none) -> C14663
- JP1: symbol Connector:USB_A -> sequencer-rescue:USB_A-Connector
- JP2: symbol Connector:Micro_SD_Card -> sequencer-rescue:Micro_SD_Card-Connector
- Q5: symbol Transistor_BJT:MMBT3904 -> sequencer-rescue:MMBT3904-Transistor_BJT; LCSC (none) -> C20526
- R10, R11, R12, R36, R49, R55, R58, R61, R67, R69, R70, R71, R72, R73, R74, R75, R77: symbol Device:R -> sequencer-rescue:R-Device
- R13: symbol Device:R -> sequencer-rescue:R-Device; LCSC (none) -> C4216
- R50: symbol Device:R -> sequencer-rescue:R-Device; LCSC (none) -> C25804
- R66: symbol Device:R -> sequencer-rescue:R-Device; LCSC (none) -> C25803
- R76: symbol Device:R -> sequencer-rescue:R-Device; LCSC (none) -> C21190
- R9: symbol Device:R -> sequencer-rescue:R-Device; LCSC (none) -> C22935
- U11: LCSC (none) -> C5613
- U12: LCSC (none) -> C5947
- U5: LCSC (none) -> C5962
Changed lines of the file:
@@
 EESchema Schematic File Version 4
 LIBS:sequencer-cache
-EELAYER 26 0
+EELAYER 30 0
 EELAYER END
 $Descr A4 11693 8268
@@
 F 5 "SN74HC165D" H 4600 4550 50  0001 C CNN "MFP"
 F 6 "SOIC-16" H 4600 4550 50  0001 C CNN "Package"
+F 7 "C5613" H 4100 5300 50  0001 C CNN "LCSC"
 	1    4100 5300
 	1    0    0    -1
@@
 F 5 "SN74HC595D" H 4600 350 50  0001 C CNN "MFP"
 F 6 "SOIC-16" H 4600 350 50  0001 C CNN "Package"
+F 7 "C5947" H 4100 1100 50  0001 C CNN "LCSC"
 	1    4100 1100
 	1    0    0    -1
@@
 $EndComp
 $Comp
-L power:GND #PWR01
+L sequencer-rescue:GND-power #PWR01
 U 1 1 59DAC8B2
 P 4000 4700
@@
 $EndComp
 $Comp
-L power:GND #PWR02
+L sequencer-rescue:GND-power #PWR02
 U 1 1 59DAC8DB
 P 4000 3300
@@
 $EndComp
 $Comp
-L power:GND #PWR03
+L sequencer-rescue:GND-power #PWR03
 U 1 1 59DAC904
 P 4000 1900
@@
 $EndComp
 $Comp
-L power:+5V #PWR04
+L sequencer-rescue:+5V-power #PWR04
 U 1 1 59DACCD2
 P 4000 1000
@@
 $EndComp
 $Comp
-L power:+5V #PWR05
+L sequencer-rescue:+5V-power #PWR05
 U 1 1 59DACCFB
 P 4000 2400
@@
 $EndComp
 $Comp
-L power:+5V #PWR06
+L sequencer-rescue:+5V-power #PWR06
 U 1 1 59DACD24
 P 4000 3800
@@
 $EndComp
 $Comp
-L Device:C C6
+L sequencer-rescue:C-Device C6
 U 1 1 59DAD327
 P 1400 5450
@@
 F 5 "GRM188R71E104JA01J" H 1425 5650 50  0001 C CNN "MFP"
 F 6 "0603" H 1425 5650 50  0001 C CNN "Package"
+F 7 "C14663" H 1400 5450 50  0001 C CNN "LCSC"
 	1    1400 5450
 	1    0    0    -1
 $EndComp
 $Comp
-L Device:C C43
+L sequencer-rescue:C-Device C43
 U 1 1 59DAD399
 P 1700 5450
@@
 $EndComp
 $Comp
-L Device:C C44
+L sequencer-rescue:C-Device C44
 U 1 1 59DAD3D5
 P 2000 5450
@@
 $EndComp
 $Comp
-L Device:C C45
+L sequencer-rescue:C-Device C45
 U 1 1 59DAD3DB
 P 2300 5450
@@
 $EndComp
 $Comp
-L power:GND #PWR07
+L sequencer-rescue:GND-power #PWR07
 U 1 1 59DADBC6
 P 4000 6100
@@
 $EndComp
 $Comp
-L power:+5V #PWR08
+L sequencer-rescue:+5V-power #PWR08
 U 1 1 59DADC53
 P 4000 5200
@@
 $EndComp
 $Comp
-L power:GND #PWR09
+L sequencer-rescue:GND-power #PWR09
 U 1 1 59DAEC89
 P 5200 6100
@@
 $EndComp
 $Comp
-L Device:C C49
+L sequencer-rescue:C-Device C49
 U 1 1 59DB526D
 P 2600 5450
@@
 $EndComp
 $Comp
-L power:+5V #PWR010
+L sequencer-rescue:+5V-power #PWR010
 U 1 1 59DB575D
 P 1300 5100
@@
 $EndComp
 $Comp
-L power:GND #PWR011
+L sequencer-rescue:GND-power #PWR011
 U 1 1 59DB5795
 P 1300 5800
@@
 $EndComp
 $Comp
-L Connector:Micro_SD_Card JP2
+L sequencer-rescue:Micro_SD_Card-Connector JP2
 U 1 1 59DC0C9C
 P 9600 1900
@@
 $EndComp
 $Comp
-L power:+3.3V #PWR012
+L sequencer-rescue:+3.3V-power #PWR012
 U 1 1 59DD8249
 P 8600 1050
@@
 $EndComp
 $Comp
-L power:GND #PWR013
+L sequencer-rescue:GND-power #PWR013
 U 1 1 59DD828A
 P 8600 2900
@@
 $EndComp
 $Comp
-L power:GND #PWR014
+L sequencer-rescue:GND-power #PWR014
 U 1 1 59DD85C7
 P 10500 2900
@@
 $EndComp
 $Comp
-L power:GND #PWR015
+L sequencer-rescue:GND-power #PWR015
 U 1 1 59DDC96B
 P 9700 5900
@@
 $EndComp
 $Comp
-L power:+3.3V #PWR016
+L sequencer-rescue:+3.3V-power #PWR016
 U 1 1 59DDCA82
 P 9600 3600
@@
 $EndComp
 $Comp
-L power:GND #PWR017
+L sequencer-rescue:GND-power #PWR017
 U 1 1 59DDD81F
 P 8400 5900
@@
 $EndComp
 $Comp
-L power:GND #PWR018
+L sequencer-rescue:GND-power #PWR018
 U 1 1 59DDDDF7
 P 7100 5900
@@
 $EndComp
 $Comp
-L Connector:USB_A JP1
+L sequencer-rescue:USB_A-Connector JP1
 U 1 1 59DE5EB2
 P 7600 3900
@@
 $EndComp
 $Comp
-L power:GND #PWR019
+L sequencer-rescue:GND-power #PWR019
 U 1 1 59E06450
 P 7600 4500
@@
 $EndComp
 $Comp
-L Device:R R50
+L sequencer-rescue:R-Device R50
 U 1 1 59E55F0E
 P 5300 5150
@@
 F 5 "ERJ-3EKF1002V" H 5250 5400 50  0001 C CNN "MFP"
 F 6 "0603" H 5250 5400 50  0001 C CNN "Package"
+F 7 "C25804" V 5300 5150 50  0001 C CNN "LCSC"
 	1    5300 5150
 	1    0    0    -1
 $EndComp
 $Comp
-L Device:R R55
+L sequencer-rescue:R-Device R55
 U 1 1 59E560D3
 P 5400 5150
@@
 $EndComp
 $Comp
-L Device:R R58
+L sequencer-rescue:R-Device R58
 U 1 1 59E56118
 P 5500 5150
@@
 $EndComp
 $Comp
-L Device:R R61
+L sequencer-rescue:R-Device R61
 U 1 1 59E56160
 P 5600 5150
@@
 $EndComp
 $Comp
-L Device:R R49
+L sequencer-rescue:R-Device R49
 U 1 1 59E561AB
 P 5700 5150
@@
 $EndComp
 $Comp
-L power:+5V #PWR020
+L sequencer-rescue:+5V-power #PWR020
 U 1 1 59E571E6
 P 6200 4700
@@
 $EndComp
 $Comp
-L Device:R R76
+L sequencer-rescue:R-Device R76
 U 1 1 59E604C8
 P 5350 2600
@@
 F 5 "ERJ-3EKF1001V" H 5300 2850 50  0001 C CNN "MFP"
 F 6 "0603" H 5300 2850 50  0001 C CNN "Package"
+F 7 "C21190" V 5350 2600 50  0001 C CNN "LCSC"
 	1    5350 2600
 	0    1    1    0
 $EndComp
 $Comp
-L Device:R R77
+L sequencer-rescue:R-Device R77
 U 1 1 59E60528
 P 5350 2500
@@
 $EndComp
 $Comp
-L Device:R R75
+L sequencer-rescue:R-Device R75
 U 1 1 59E60C94
 P 5350 2700
@@
 $EndComp
 $Comp
-L Device:R R74
+L sequencer-rescue:R-Device R74
 U 1 1 59E60F5A
 P 5350 2800
@@
 $EndComp
 $Comp
-L Device:R R70
+L sequencer-rescue:R-Device R70
 U 1 1 59E61471
 P 5350 3200
@@
 $EndComp
 $Comp
-L Device:R R71
+L sequencer-rescue:R-Device R71
 U 1 1 59E6153A
 P 5350 3100
@@
 $EndComp
 $Comp
-L Device:R R72
+L sequencer-rescue:R-Device R72
 U 1 1 59E61584
 P 5350 3000
@@
 $EndComp
 $Comp
-L Device:R R73
+L sequencer-rescue:R-Device R73
 U 1 1 59E6158A
 P 5350 2900
@@
 F 5 "SN74HCT125D" H 1600 1000 60  0001 C CNN "MFP"
 F 6 "SOIC-14" H 2100 50  50  0001 C CNN "Package"
+F 7 "C5962" H 1600 1000 50  0001 C CNN "LCSC"
 	1    1600 1000
 	1    0    0    -1
 $EndComp
 $Comp
-L power:GND #PWR021
+L sequencer-rescue:GND-power #PWR021
 U 1 1 59E5F67D
 P 1500 2000
@@
 $EndComp
 $Comp
-L power:+5V #PWR022
+L sequencer-rescue:+5V-power #PWR022
 U 1 1 59E5F6E5
 P 1500 900
@@
 $EndComp
 $Comp
-L Device:R R13
+L sequencer-rescue:R-Device R13
 U 1 1 5AEA4C2A
 P 8400 1350
@@
 F 5 "ERJ-3EKF3302V" H 8480 1450 50  0001 C CNN "MFP"
 F 6 "0603" H 8480 1450 50  0001 C CNN "Package"
+F 7 "C4216" V 8400 1350 50  0001 C CNN "LCSC"
 	1    8400 1350
 	-1   0    0    1
 $EndComp
 $Comp
-L Device:R R9
+L sequencer-rescue:R-Device R9
 U 1 1 5AEA4CDA
 P 8400 2550
@@
 F 5 "ERJ-3EKF1004V" H 8480 2650 50  0001 C CNN "MFP"
 F 6 "0603" H 8480 2650 50  0001 C CNN "Package"
+F 7 "C22935" V 8400 2550 50  0001 C CNN "LCSC"
 	1    8400 2550
 	-1   0    0    1
 $EndComp
 $Comp
-L Device:R R10
+L sequencer-rescue:R-Device R10
 U 1 1 5AEA4D5E
 P 7800 1350
@@
 $EndComp
 $Comp
-L Device:R R11
+L sequencer-rescue:R-Device R11
 U 1 1 5AEA4DC8
 P 8000 1350
@@
 $EndComp
 $Comp
-L Device:R R12
+L sequencer-rescue:R-Device R12
 U 1 1 5AEA93F2
 P 8200 1350
@@
 $EndComp
 $Comp
-L Device:R R36
+L sequencer-rescue:R-Device R36
 U 1 1 5AEB2AD1
 P 9500 5550
@@
 $EndComp
 $Comp
-L Transistor_BJT:MMBT3904 Q5
+L sequencer-rescue:MMBT3904-Transistor_BJT Q5
 U 1 1 5AEB9A70
 P 2600 2900
@@
 F 5 "MMBT3904LT1G" H 2800 3075 50  0001 C CNN "MFP"
 F 6 "SOT-23" H 2800 3075 50  0001 C CNN "Package"
+F 7 "C20526" H 2600 2900 50  0001 C CNN "LCSC"
 	1    2600 2900
 	1    0    0    -1
 $EndComp
 $Comp
-L Device:R R67
+L sequencer-rescue:R-Device R67
 U 1 1 5AEB9A79
 P 2700 2350
@@
 $EndComp
 $Comp
-L power:GND #PWR023
+L sequencer-rescue:GND-power #PWR023
 U 1 1 5AEB9A80
 P 2700 3500
@@
 $EndComp
 $Comp
-L power:+5V #PWR024
+L sequencer-rescue:+5V-power #PWR024
 U 1 1 5AEB9A86
 P 2700 2100
@@
 $EndComp
 $Comp
-L Device:R R66
+L sequencer-rescue:R-Device R66
 U 1 1 5AEBCC66
 P 2050 2900
@@
 F 5 "ERJ-3EKF1002V" H 2130 3000 50  0001 C CNN "MFP"
 F 6 "0603" H 2130 3000 50  0001 C CNN "Package"
+F 7 "C25803" V 2050 2900 50  0001 C CNN "LCSC"
 	1    2050 2900
 	0    1    1    0
 $EndComp
 $Comp
-L Device:R R69
+L sequencer-rescue:R-Device R69
 U 1 1 5AEBCE61
 P 2300 3150

Commit message: Fixed LCSC values.
Parts:
- R66: LCSC C25803 -> (none)
Changed lines of the file:
@@
 EESchema Schematic File Version 4
-LIBS:sequencer-cache
 EELAYER 30 0
 EELAYER END
@@
 F 5 "ERJ-3EKF1002V" H 2130 3000 50  0001 C CNN "MFP"
 F 6 "0603" H 2130 3000 50  0001 C CNN "Package"
-F 7 "C25803" V 2050 2900 50  0001 C CNN "LCSC"
 	1    2050 2900
 	0    1    1    0
@@
 	4100 5900 4000 5900
 Wire Wire Line
-	3700 5500 4100 5500
-Wire Wire Line
-	3700 5700 4100 5700
-Wire Wire Line
 	5100 5300 5300 5300
 Wire Wire Line
@@
 Wire Wire Line
 	2700 3400 2700 3500
+Wire Wire Line
+	3700 5700 4100 5700
+Wire Wire Line
+	3700 5500 4100 5500
 $EndSCHEMATC
