File: global.sch (KiCad schematic (older format))
At the start: 37 parts, among them Q5 MMBT3904, U11 74HC165, U12 74HC595, U13 74HC595, U14 74HC595, U5 74HCT125

Commit message: Some cleanup. Frontpanel with Copper Labels.
Parts:
- R66: LCSC C25803 -> (none)
- R69: LCSC (none) -> C25803
Changed lines of the file:
@@
 F 5 "ERJ-3EKF1002V" H 2130 3000 50  0001 C CNN "MFP"
 F 6 "0603" H 2130 3000 50  0001 C CNN "Package"
-F 7 "C25803" V 2050 2900 50  0001 C CNN "LCSC"
 	1    2050 2900
 	0    1    1    0
@@
 F 5 "ERJ-3EKF1003V" H 2380 3250 50  0001 C CNN "MFP"
 F 6 "0603" H 2380 3250 50  0001 C CNN "Package"
+F 7 "C25803" V 2300 3150 50  0001 C CNN "LCSC"
 	1    2300 3150
 	1    0    0    -1
