File: led-matrix.sch (KiCad schematic (older format))
At the start: 32 parts

Commit message: Added JCLC part numbers.
Parts:
- LED1, LED10, LED11, LED12, LED13, LED14, LED15, LED16, LED17, LED18, LED19, LED2, LED20, LED21, LED22, LED23, LED24, LED25, LED26, LED27, LED28, LED29, LED3, LED30, LED31, LED32, LED4, LED5, LED6, LED7, LED8, LED9: symbol Device:LED_Dual_ACA -> sequencer-rescue:LED_Dual_ACA-Device
Changed lines of the file:
@@
 EESchema Schematic File Version 4
 LIBS:sequencer-cache
-EELAYER 26 0
+EELAYER 30 0
 EELAYER END
 $Descr A4 11693 8268
@@
 $EndDescr
 $Comp
-L Device:LED_Dual_ACA LED1
+L sequencer-rescue:LED_Dual_ACA-Device LED1
 U 1 1 59DAB354
 P 2400 1900
@@
 $EndComp
 $Comp
-L Device:LED_Dual_ACA LED5
+L sequencer-rescue:LED_Dual_ACA-Device LED5
 U 1 1 59DAB3C2
 P 2400 2700
@@
 $EndComp
 $Comp
-L Device:LED_Dual_ACA LED15
+L sequencer-rescue:LED_Dual_ACA-Device LED15
 U 1 1 59DAB418
 P 2400 3500
@@
 $EndComp
 $Comp
-L Device:LED_Dual_ACA LED25
+L sequencer-rescue:LED_Dual_ACA-Device LED25
 U 1 1 59DAB41E
 P 2400 4300
@@
 $EndComp
 $Comp
-L Device:LED_Dual_ACA LED2
+L sequencer-rescue:LED_Dual_ACA-Device LED2
 U 1 1 59DAB4C6
 P 3300 1900
@@
 $EndComp
 $Comp
-L Device:LED_Dual_ACA LED6
+L sequencer-rescue:LED_Dual_ACA-Device LED6
 U 1 1 59DAB4CC
 P 3300 2700
@@
 $EndComp
 $Comp
-L Device:LED_Dual_ACA LED16
+L sequencer-rescue:LED_Dual_ACA-Device LED16
 U 1 1 59DAB4D2
 P 3300 3500
@@
 $EndComp
 $Comp
-L Device:LED_Dual_ACA LED26
+L sequencer-rescue:LED_Dual_ACA-Device LED26
 U 1 1 59DAB4D8
 P 3300 4300
@@
 $EndComp
 $Comp
-L Device:LED_Dual_ACA LED3
+L sequencer-rescue:LED_Dual_ACA-Device LED3
 U 1 1 59DAB5EE
 P 4200 1900
@@
 $EndComp
 $Comp
-L Device:LED_Dual_ACA LED7
+L sequencer-rescue:LED_Dual_ACA-Device LED7
 U 1 1 59DAB5F4
 P 4200 2700
@@
 $EndComp
 $Comp
-L Device:LED_Dual_ACA LED17
+L sequencer-rescue:LED_Dual_ACA-Device LED17
 U 1 1 59DAB5FA
 P 4200 3500
@@
 $EndComp
 $Comp
-L Device:LED_Dual_ACA LED27
+L sequencer-rescue:LED_Dual_ACA-Device LED27
 U 1 1 59DAB600
 P 4200 4300
@@
 $EndComp
 $Comp
-L Device:LED_Dual_ACA LED4
+L sequencer-rescue:LED_Dual_ACA-Device LED4
 U 1 1 59DAB606
 P 5100 1900
@@
 $EndComp
 $Comp
-L Device:LED_Dual_ACA LED8
+L sequencer-rescue:LED_Dual_ACA-Device LED8
 U 1 1 59DAB60C
 P 5100 2700
@@
 $EndComp
 $Comp
-L Device:LED_Dual_ACA LED18
+L sequencer-rescue:LED_Dual_ACA-Device LED18
 U 1 1 59DAB612
 P 5100 3500
@@
 $EndComp
 $Comp
-L Device:LED_Dual_ACA LED28
+L sequencer-rescue:LED_Dual_ACA-Device LED28
 U 1 1 59DAB618
 P 5100 4300
@@
 $EndComp
 $Comp
-L Device:LED_Dual_ACA LED13
+L sequencer-rescue:LED_Dual_ACA-Device LED13
 U 1 1 59DAB7AE
 P 6000 1900
@@
 $EndComp
 $Comp
-L Device:LED_Dual_ACA LED9
+L sequencer-rescue:LED_Dual_ACA-Device LED9
 U 1 1 59DAB7B4
 P 6000 2700
@@
 $EndComp
 $Comp
-L Device:LED_Dual_ACA LED19
+L sequencer-rescue:LED_Dual_ACA-Device LED19
 U 1 1 59DAB7BA
 P 6000 3500
@@
 $EndComp
 $Comp
-L Device:LED_Dual_ACA LED29
+L sequencer-rescue:LED_Dual_ACA-Device LED29
 U 1 1 59DAB7C0
 P 6000 4300
@@
 $EndComp
 $Comp
-L Device:LED_Dual_ACA LED14
+L sequencer-rescue:LED_Dual_ACA-Device LED14
 U 1 1 59DAB7C6
 P 6900 1900
@@
 $EndComp
 $Comp
-L Device:LED_Dual_ACA LED10
+L sequencer-rescue:LED_Dual_ACA-Device LED10
 U 1 1 59DAB7CC
 P 6900 2700
@@
 $EndComp
 $Comp
-L Device:LED_Dual_ACA LED20
+L sequencer-rescue:LED_Dual_ACA-Device LED20
 U 1 1 59DAB7D2
 P 6900 3500
@@
 $EndComp
 $Comp
-L Device:LED_Dual_ACA LED30
+L sequencer-rescue:LED_Dual_ACA-Device LED30
 U 1 1 59DAB7D8
 P 6900 4300
@@
 $EndComp
 $Comp
-L Device:LED_Dual_ACA LED23
+L sequencer-rescue:LED_Dual_ACA-Device LED23
 U 1 1 59DAB7DE
 P 7800 1900
@@
 $EndComp
 $Comp
-L Device:LED_Dual_ACA LED11
+L sequencer-rescue:LED_Dual_ACA-Device LED11
 U 1 1 59DAB7E4
 P 7800 2700
@@
 $EndComp
 $Comp
-L Device:LED_Dual_ACA LED21
+L sequencer-rescue:LED_Dual_ACA-Device LED21
 U 1 1 59DAB7EA
 P 7800 3500
@@
 $EndComp
 $Comp
-L Device:LED_Dual_ACA LED31
+L sequencer-rescue:LED_Dual_ACA-Device LED31
 U 1 1 59DAB7F0
 P 7800 4300
@@
 $EndComp
 $Comp
-L Device:LED_Dual_ACA LED24
+L sequencer-rescue:LED_Dual_ACA-Device LED24
 U 1 1 59DAB7F6
 P 8700 1900
@@
 $EndComp
 $Comp
-L Device:LED_Dual_ACA LED12
+L sequencer-rescue:LED_Dual_ACA-Device LED12
 U 1 1 59DAB7FC
 P 8700 2700
@@
 $EndComp
 $Comp
-L Device:LED_Dual_ACA LED22
+L sequencer-rescue:LED_Dual_ACA-Device LED22
 U 1 1 59DAB802
 P 8700 3500
@@
 $EndComp
 $Comp
-L Device:LED_Dual_ACA LED32
+L sequencer-rescue:LED_Dual_ACA-Device LED32
 U 1 1 59DAB808
 P 8700 4300
