File: mcu.sch (KiCad schematic (older format))
At the start: 18 parts, among them SW19 EVQQ2, SW8 EVQQ2, U9 STM32F405RGTx, Y1 8MHz

Commit message: Added JCLC part numbers.
Parts:
- C17, C18, C20, C23, C30, C32, C36, C42: symbol Device:C -> sequencer-rescue:C-Device
- C39: symbol Device:C -> sequencer-rescue:C-Device; LCSC (none) -> C15849
- C41: symbol Device:C -> sequencer-rescue:C-Device; LCSC (none) -> C1647
- JP4: symbol Connector_Generic:Conn_02x05_Odd_Even -> sequencer-rescue:Conn_02x05_Odd_Even-Connector_Generic
- JP6: symbol Connector_Generic:Conn_01x06 -> sequencer-rescue:Conn_01x06-Connector_Generic
- R79, R82: symbol Device:R -> sequencer-rescue:R-Device
- SW19, SW8: symbol Switch:SW_Push -> sequencer-rescue:SW_Push-Switch
- U9: LCSC (none) -> C15742
- Y1: symbol Device:Crystal -> sequencer-rescue:Crystal-Device
Changed lines of the file:
@@
 EESchema Schematic File Version 4
 LIBS:sequencer-cache
-EELAYER 26 0
+EELAYER 30 0
 EELAYER END
 $Descr A4 11693 8268
@@
 F 5 "STM32F405RGT6" H 1600 5225 50  0001 C CNN "MFP"
 F 6 "LQFP-64" H 1600 5225 50  0001 C CNN "Package"
+F 7 "C15742" H 5800 3200 50  0001 C CNN "LCSC"
 	1    5800 3200
 	1    0    0    -1
 $EndComp
 $Comp
-L Connector_Generic:Conn_01x06 JP6
+L sequencer-rescue:Conn_01x06-Connector_Generic JP6
 U 1 1 59DB9577
 P 3400 6800
@@
 $EndComp
 $Comp
-L power:GND #PWR055
+L sequencer-rescue:GND-power #PWR055
 U 1 1 59DB9615
 P 3700 7100
@@
 $EndComp
 $Comp
-L Connector_Generic:Conn_02x05_Odd_Even JP4
+L sequencer-rescue:Conn_02x05_Odd_Even-Connector_Generic JP4
 U 1 1 59DB9B82
 P 1400 6800
@@
 $EndComp
 $Comp
-L power:+3.3V #PWR056
+L sequencer-rescue:+3.3V-power #PWR056
 U 1 1 59DB9CCC
 P 1100 6500
@@
 $EndComp
 $Comp
-L power:GND #PWR057
+L sequencer-rescue:GND-power #PWR057
 U 1 1 59DB9CF4
 P 1100 7100
@@
 $EndComp
 $Comp
-L power:+3.3V #PWR058
+L sequencer-rescue:+3.3V-power #PWR058
 U 1 1 59DB9EAC
 P 5500 1000
@@
 $EndComp
 $Comp
-L power:+3.3VA #PWR059
+L sequencer-rescue:+3.3VA-power #PWR059
 U 1 1 59DB9EE7
 P 6000 1000
@@
 $EndComp
 $Comp
-L power:GND #PWR060
+L sequencer-rescue:GND-power #PWR060
 U 1 1 59DB9FE7
 P 5800 5400
@@
 $EndComp
 $Comp
-L Device:Crystal Y1
+L sequencer-rescue:Crystal-Device Y1
 U 1 1 59DBA308
 P 7500 5750
@@
 $EndComp
 $Comp
-L Device:C C41
+L sequencer-rescue:C-Device C41
 U 1 1 59DBA373
 P 7250 5500
@@
 F 5 "GRM1885C1H180JA01J" H 7275 5700 50  0001 C CNN "MFP"
 F 6 "0603" H 7275 5700 50  0001 C CNN "Package"
+F 7 "C1647" H 7250 5500 50  0001 C CNN "LCSC"
 	1    7250 5500
 	0    -1   -1   0
 $EndComp
 $Comp
-L Device:C C42
+L sequencer-rescue:C-Device C42
 U 1 1 59DBA3A0
 P 7250 6000
@@
 $EndComp
 $Comp
-L power:GND #PWR061
+L sequencer-rescue:GND-power #PWR061
 U 1 1 59DBA437
 P 7000 6100
@@
 $EndComp
 $Comp
-L Device:C C23
+L sequencer-rescue:C-Device C23
 U 1 1 59DBB4BE
 P 1150 2050
@@
 $EndComp
 $Comp
-L Device:C C18
+L sequencer-rescue:C-Device C18
 U 1 1 59DBB504
 P 1150 2250
@@
 $EndComp
 $Comp
-L power:GND #PWR062
+L sequencer-rescue:GND-power #PWR062
 U 1 1 59DBB736
 P 800 2250
@@
 $EndComp
 $Comp
-L Switch:SW_Push SW19
+L sequencer-rescue:SW_Push-Switch SW19
 U 1 1 59DD439D
 P 5800 6400
@@
 $EndComp
 $Comp
-L Switch:SW_Push SW8
+L sequencer-rescue:SW_Push-Switch SW8
 U 1 1 59DD44E7
 P 5200 6900
@@
 $EndComp
 $Comp
-L Device:R R82
+L sequencer-rescue:R-Device R82
 U 1 1 59DD490D
 P 5200 6350
@@
 $EndComp
 $Comp
-L Device:R R79
+L sequencer-rescue:R-Device R79
 U 1 1 59DD4953
 P 5800 6950
@@
 $EndComp
 $Comp
-L power:+3.3V #PWR063
+L sequencer-rescue:+3.3V-power #PWR063
 U 1 1 59DD49A9
 P 5200 6100
@@
 $EndComp
 $Comp
-L power:+3.3V #PWR064
+L sequencer-rescue:+3.3V-power #PWR064
 U 1 1 59DD49E1
 P 5800 6100
@@
 $EndComp
 $Comp
-L power:GND #PWR065
+L sequencer-rescue:GND-power #PWR065
 U 1 1 59DD4A83
 P 5200 7200
@@
 $EndComp
 $Comp
-L power:GND #PWR066
+L sequencer-rescue:GND-power #PWR066
 U 1 1 59DD4ABB
 P 5800 7200
@@
 $EndComp
 $Comp
-L Device:C C30
+L sequencer-rescue:C-Device C30
 U 1 1 59E34530
 P 8600 5750
@@
 $EndComp
 $Comp
-L Device:C C32
+L sequencer-rescue:C-Device C32
 U 1 1 59E345BC
 P 8900 5750
@@
 $EndComp
 $Comp
-L Device:C C20
+L sequencer-rescue:C-Device C20
 U 1 1 59E34607
 P 9200 5750
@@
 $EndComp
 $Comp
-L Device:C C17
+L sequencer-rescue:C-Device C17
 U 1 1 59E34648
 P 9500 5750
@@
 $EndComp
 $Comp
-L power:+3.3V #PWR067
+L sequencer-rescue:+3.3V-power #PWR067
 U 1 1 59E34B90
 P 8500 5400
@@
 $EndComp
 $Comp
-L power:GND #PWR068
+L sequencer-rescue:GND-power #PWR068
 U 1 1 59E34BD4
 P 8500 6100
@@
 $EndComp
 $Comp
-L power:+3.3VA #PWR069
+L sequencer-rescue:+3.3VA-power #PWR069
 U 1 1 59E35078
 P 9900 5400
@@
 $EndComp
 $Comp
-L power:GND #PWR070
+L sequencer-rescue:GND-power #PWR070
 U 1 1 59E350BC
 P 9900 6100
@@
 $EndComp
 $Comp
-L Device:C C39
+L sequencer-rescue:C-Device C39
 U 1 1 59E35219
 P 10000 5750
@@
 F 5 "GRM188R61A105KA61J" H 10025 5950 50  0001 C CNN "MFP"
 F 6 "0603" H 10025 5950 50  0001 C CNN "Package"
+F 7 "C15849" H 10000 5750 50  0001 C CNN "LCSC"
 	1    10000 5750
 	1    0    0    -1
 $EndComp
 $Comp
-L Device:C C36
+L sequencer-rescue:C-Device C36
 U 1 1 59E3526B
 P 10300 5750
@@
 $EndComp
 $Comp
-L power:PWR_FLAG #FLG071
+L sequencer-rescue:PWR_FLAG-power #FLG071
 U 1 1 59F48B1D
 P 1400 2300
@@
 $EndComp
 $Comp
-L power:PWR_FLAG #FLG072
+L sequencer-rescue:PWR_FLAG-power #FLG072
 U 1 1 59F48C86
 P 1400 2000
