File: power.sch (KiCad schematic (older format))
At the start: 24 parts, among them U10 LM1117-3.3, U16 R-78E5.0-1.0, U3 STMPS2151, U7 LM1117-3.3

Commit message: Added JCLC part numbers.
Parts:
- C1, C14, C19, C2, C31, C35, C8: symbol Device:C -> sequencer-rescue:C-Device
- C13, C24, C40, C46, C5: symbol Device:CP1 -> sequencer-rescue:CP1-Device
- D1: symbol Device:D_Schottky_ALT -> sequencer-rescue:D_Schottky_ALT-Device
- D3: symbol Device:D -> sequencer-rescue:D-Device; LCSC (none) -> C117948
- D4: symbol Device:D -> sequencer-rescue:D-Device
- JP5: symbol Connector_Generic:Conn_02x05_Odd_Even -> sequencer-rescue:Conn_02x05_Odd_Even-Connector_Generic
- L1: symbol Device:Ferrite_Bead -> sequencer-rescue:Ferrite_Bead-Device; LCSC (none) -> C1002
- L2: symbol Device:Ferrite_Bead -> sequencer-rescue:Ferrite_Bead-Device
- R5, R8: symbol Device:R -> sequencer-rescue:R-Device
- U10, U7: symbol Regulator_Linear:LM1117-3.3 -> sequencer-rescue:LM1117-3.3-Regulator_Linear
Changed lines of the file:
@@
 EESchema Schematic File Version 4
 LIBS:sequencer-cache
-EELAYER 26 0
+EELAYER 30 0
 EELAYER END
 $Descr A4 11693 8268
@@
 $EndDescr
 $Comp
-L power:+12V #PWR025
+L sequencer-rescue:+12V-power #PWR025
 U 1 1 59ADCE23
 P 900 1200
@@
 $EndComp
 $Comp
-L power:-12V #PWR035
+L sequencer-rescue:-12V-power #PWR035
 U 1 1 59ADCE37
 P 900 1800
@@
 $EndComp
 $Comp
-L Connector_Generic:Conn_02x05_Odd_Even JP5
+L sequencer-rescue:Conn_02x05_Odd_Even-Connector_Generic JP5
 U 1 1 59ADD000
 P 1700 1500
@@
 $EndComp
 $Comp
-L Device:D D3
+L sequencer-rescue:D-Device D3
 U 1 1 59ADD0E1
 P 1150 1300
@@
 F 5 "1N5819HW-7-F" H 1150 1500 50  0001 C CNN "MFP"
 F 6 "SOD-123" H 1150 1500 50  0001 C CNN "Package"
+F 7 "C117948" H 1150 1300 50  0001 C CNN "LCSC"
 	1    1150 1300
 	1    0    0    -1
 $EndComp
 $Comp
-L Device:D D4
+L sequencer-rescue:D-Device D4
 U 1 1 59ADD164
 P 1150 1700
@@
 $EndComp
 $Comp
-L power:GND #PWR026
+L sequencer-rescue:GND-power #PWR026
 U 1 1 59ADD2AE
 P 2300 1600
@@
 $EndComp
 $Comp
-L Device:CP1 C13
+L sequencer-rescue:CP1-Device C13
 U 1 1 59ADD50C
 P 3000 1250
@@
 $EndComp
 $Comp
-L power:-12V #PWR048
+L sequencer-rescue:-12V-power #PWR048
 U 1 1 59ADD571
 P 3000 2000
@@
 $EndComp
 $Comp
-L power:+12V #PWR027
+L sequencer-rescue:+12V-power #PWR027
 U 1 1 59ADD597
 P 3000 1000
@@
 $EndComp
 $Comp
-L power:GND #PWR028
+L sequencer-rescue:GND-power #PWR028
 U 1 1 59ADD670
 P 2800 1600
@@
 $EndComp
 $Comp
-L Regulator_Linear:LM1117-3.3 U7
+L sequencer-rescue:LM1117-3.3-Regulator_Linear U7
 U 1 1 59DEB84A
 P 7300 1300
@@
 $EndComp
 $Comp
-L Device:Ferrite_Bead L1
+L sequencer-rescue:Ferrite_Bead-Device L1
 U 1 1 59DEC32E
 P 6550 1300
@@
 F 5 "MI0603K300R-10" H 6550 1300 60  0001 C CNN "MFP"
 F 6 "0603" H 6400 1425 50  0001 C CNN "Package"
+F 7 "C1002" V 6550 1300 50  0001 C CNN "LCSC"
 	1    6550 1300
 	0    1    1    0
 $EndComp
 $Comp
-L Device:CP1 C24
+L sequencer-rescue:CP1-Device C24
 U 1 1 59DEC56E
 P 7800 1550
@@
 $EndComp
 $Comp
-L Device:C C14
+L sequencer-rescue:C-Device C14
 U 1 1 59DEC574
 P 8100 1550
@@
 $EndComp
 $Comp
-L power:GND #PWR029
+L sequencer-rescue:GND-power #PWR029
 U 1 1 59DEC57A
 P 6800 1800
@@
 $EndComp
 $Comp
-L power:GND #PWR030
+L sequencer-rescue:GND-power #PWR030
 U 1 1 59DEC580
 P 7800 1800
@@
 $EndComp
 $Comp
-L power:GND #PWR031
+L sequencer-rescue:GND-power #PWR031
 U 1 1 59DEC586
 P 8100 1800
@@
 $EndComp
 $Comp
-L power:+3V3 #PWR032
+L sequencer-rescue:+3V3-power #PWR032
 U 1 1 59DEC592
 P 8100 1200
@@
 $EndComp
 $Comp
-L power:GND #PWR033
+L sequencer-rescue:GND-power #PWR033
 U 1 1 59DEC598
 P 7300 1800
@@
 $EndComp
 $Comp
-L Regulator_Linear:LM1117-3.3 U10
+L sequencer-rescue:LM1117-3.3-Regulator_Linear U10
 U 1 1 59DEC7FA
 P 9800 1300
@@
 $EndComp
 $Comp
-L Device:C C31
+L sequencer-rescue:C-Device C31
 U 1 1 59DEC80C
 P 10600 1550
@@
 $EndComp
 $Comp
-L power:GND #PWR034
+L sequencer-rescue:GND-power #PWR034
 U 1 1 59DEC812
 P 9300 1800
@@
 $EndComp
 $Comp
-L power:GND #PWR0116
+L sequencer-rescue:GND-power #PWR0116
 U 1 1 59DEC818
 P 10300 1800
@@
 $EndComp
 $Comp
-L power:GND #PWR036
+L sequencer-rescue:GND-power #PWR036
 U 1 1 59DEC81E
 P 10600 1800
@@
 $EndComp
 $Comp
-L power:GND #PWR037
+L sequencer-rescue:GND-power #PWR037
 U 1 1 59DEC82A
 P 9800 1800
@@
 $EndComp
 $Comp
-L power:+12V #PWR038
+L sequencer-rescue:+12V-power #PWR038
 U 1 1 59DECCAB
 P 3900 1200
@@
 $EndComp
 $Comp
-L power:+3.3VA #PWR039
+L sequencer-rescue:+3.3VA-power #PWR039
 U 1 1 59DED3E1
 P 10600 1200
@@
 $EndComp
 $Comp
-L Device:C C2
+L sequencer-rescue:C-Device C2
 U 1 1 59DED9C5
 P 5600 1550
@@
 $EndComp
 $Comp
-L power:GND #PWR040
+L sequencer-rescue:GND-power #PWR040
 U 1 1 59DED9CB
 P 4200 1800
@@
 $EndComp
 $Comp
-L power:GND #PWR041
+L sequencer-rescue:GND-power #PWR041
 U 1 1 59DED9D1
 P 5300 1800
@@
 $EndComp
 $Comp
-L power:GND #PWR042
+L sequencer-rescue:GND-power #PWR042
 U 1 1 59DED9D7
 P 5600 1800
@@
 $EndComp
 $Comp
-L power:GND #PWR043
+L sequencer-rescue:GND-power #PWR043
 U 1 1 59DED9DD
 P 4750 1800
@@
 $EndComp
 $Comp
-L power:+5V #PWR044
+L sequencer-rescue:+5V-power #PWR044
 U 1 1 59DEDB3A
 P 5600 1200
@@
 $EndComp
 $Comp
-L Device:D_Schottky_ALT D1
+L sequencer-rescue:D_Schottky_ALT-Device D1
 U 1 1 59DF06B3
 P 4600 3250
@@
 $EndComp
 $Comp
-L power:-12V #PWR050
+L sequencer-rescue:-12V-power #PWR050
 U 1 1 59DF1046
 P 4000 2900
@@
 $EndComp
 $Comp
-L Device:R R8
+L sequencer-rescue:R-Device R8
 U 1 1 59DF10B1
 P 4250 3000
@@
 $EndComp
 $Comp
-L Device:C C1
+L sequencer-rescue:C-Device C1
 U 1 1 59DF1870
 P 4900 3250
@@
 $EndComp
 $Comp
-L power:GND #PWR045
+L sequencer-rescue:GND-power #PWR045
 U 1 1 59DF1FC9
 P 4600 3600
@@
 $EndComp
 $Comp
-L power:+5V #PWR046
+L sequencer-rescue:+5V-power #PWR046
 U 1 1 59DFDC6E
 P 1600 2900
@@
 $EndComp
 $Comp
-L power:GND #PWR047
+L sequencer-rescue:GND-power #PWR047
 U 1 1 59DFDCE5
 P 1600 3600
@@
 $EndComp
 $Comp
-L Device:R R5
+L sequencer-rescue:R-Device R5
 U 1 1 59E00C96
 P 1400 3350
@@
 $EndComp
 $Comp
-L power:GND #PWR0118
+L sequencer-rescue:GND-power #PWR0118
 U 1 1 59E00E5E
 P 1400 3600
@@
 $EndComp
 $Comp
-L Device:CP1 C46
+L sequencer-rescue:CP1-Device C46
 U 1 1 59E0E120
 P 3000 1750
@@
 $EndComp
 $Comp
-L Device:CP1 C40
+L sequencer-rescue:CP1-Device C40
 U 1 1 59E0FE4F
 P 10300 1550
@@
 $EndComp
 $Comp
-L Device:CP1 C5
+L sequencer-rescue:CP1-Device C5
 U 1 1 59E0FEB0
 P 5300 1550
@@
 $EndComp
 $Comp
-L Device:Ferrite_Bead L2
+L sequencer-rescue:Ferrite_Bead-Device L2
 U 1 1 59E11A13
 P 9050 1300
@@
 $EndComp
 $Comp
-L Device:C C19
+L sequencer-rescue:C-Device C19
 U 1 1 59E52EDD
 P 6800 1550
@@
 $EndComp
 $Comp
-L Device:C C35
+L sequencer-rescue:C-Device C35
 U 1 1 59E53513
 P 9300 1550
@@
 $EndComp
 $Comp
-L Device:C C8
+L sequencer-rescue:C-Device C8
 U 1 1 59E535E8
 P 4200 1550
@@
 $EndComp
 $Comp
-L power:PWR_FLAG #FLG049
+L sequencer-rescue:PWR_FLAG-power #FLG049
 U 1 1 59F34CFD
 P 6800 1200
@@
 $EndComp
 $Comp
-L power:PWR_FLAG #FLG050
+L sequencer-rescue:PWR_FLAG-power #FLG050
 U 1 1 59F34D75
 P 9300 1200
@@
 $EndComp
 $Comp
-L power:+5V #PWR051
+L sequencer-rescue:+5V-power #PWR051
 U 1 1 5AEF8A3B
 P 6300 1200
@@
 $EndComp
 $Comp
-L power:PWR_FLAG #FLG052
+L sequencer-rescue:PWR_FLAG-power #FLG052
 U 1 1 5BBB58DA
 P 2100 1200
@@
 $EndComp
 $Comp
-L power:PWR_FLAG #FLG053
+L sequencer-rescue:PWR_FLAG-power #FLG053
 U 1 1 5BBB5936
 P 2100 1800
@@
 $EndComp
 $Comp
-L power:+5V #PWR054
+L sequencer-rescue:+5V-power #PWR054
 U 1 1 5BBB67BF
 P 8800 1200
